File: kicad_proj1st/kicad_proj1st.kicad_pcb (KiCad board)
At the start: 4 copper layers, 58 x 52.5 mm, 41 parts, among them J1 Conn_01x02, J2 Conn_01x05, J3 Conn_01x02, J4 Conn_01x02, J5 Conn_01x02, J6 Conn_01x02, J7 Conn_01x06, Q1 TSM2302CX, Q2 TSM2302CX, Q3 TSM2302CX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

Commit message: Prototype 2 fin?
Parts:
- C5: value .1uC -> .1uF
- C6: value 4.7uC -> 4.7uF
- moved R11 60.0 mm to (70.2, 71.0), turned to 0 degrees
- moved L1 59.9 mm to (66.2, 83.5), turned to 180 degrees
- moved J6 58.1 mm to (66.0, 93.2), turned to 90 degrees
- moved Q4 53.6 mm to (71.5, 91.2), turned to 180 degrees
- moved R10 49.2 mm to (70.2, 73.8), turned to 180 degrees
- moved R4 48.9 mm to (72.8, 95.5), turned to 180 degrees
- moved R9 48.8 mm to (70.7, 75.5), turned to 0 degrees
- moved J2 39.3 mm to (60.0, 59.8), turned to 0 degrees
- moved R2 35.7 mm to (94.8, 53.0), turned to -90 degrees
- moved C2 34.4 mm to (99.5, 62.8), turned to 90 degrees
- moved C4 34.1 mm to (97.2, 72.3), turned to -90 degrees
- moved C3 31.9 mm to (102.2, 69.5), turned to 90 degrees
- moved C8 30.4 mm to (64.3, 78.2), turned to 180 degrees
- moved Q2 29.7 mm to (95.8, 56.5), turned to 0 degrees
- moved U1 29.5 mm to (98.5, 67.5)
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Routing:
- net Net-(U3-SW): track 159.8 -> 28.5 mm, vias 6 -> 0
- net Net-(U3-COMP): track 98.4 -> 7.47 mm, vias 5 -> 0
- net Net-(U3-FB): track 83.0 -> 4.45 mm, vias 4 -> 0
- net Net-(C12-Pad1): track 76.9 -> 2.05 mm, vias 4 -> 0
- net CH4: track 84.2 -> 19.7 mm, vias 6 -> 1
- net SDA: track 100.1 -> 162.8 mm, vias 8 -> 11
- net CH3: track 76.3 -> 16.3 mm, vias 4 -> 1
- net CH2: track 77.8 -> 17.9 mm, vias 5 -> 1
- net V_OUT: track 122.6 -> 78.8 mm, vias 7 -> 1
- net SCL: track 112.9 -> 150.7 mm, vias 8 -> 10
- net /Motor Switch2: track 64.9 -> 30.6 mm
- net Net-(U3-ILIM): track 35.7 -> 2.70 mm, vias 4 -> 0
- net Net-(U3-FSW): track 25.9 -> 2.69 mm, vias 4 -> 0
- net Net-(U3-VCC): track 22.7 -> 3.20 mm, vias 2 -> 0
- net CH1: track 54.1 -> 36.4 mm, vias 6 -> 3
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Other:
- board size 58 x 52.5 mm -> 50 x 50 mm
- board text added: "Muhammad Ali"
- board text removed: "3v3"
- board text removed: "CH1"
- board text removed: "GND"
- board text removed: "Muhammad Ali V2.1"
- board text removed: "RFE8V"
- board text removed: "SCL"
- board text removed: "SDA"
- board text removed: "VBAT"
- board text removed: "VOUT"

Commit message: update
Parts:
- added J8: Conn_01x01, Connector_PinHeader_2.54mm:PinHeader_1x01_P2.54mm_Vertical, F.Cu at (105.0, 58.5)
- moved J4 2.00 mm to (101.5, 51.8)
Routing:
- net GND: track 0.00 -> 2.03 mm, vias 1 -> 17
- net /Motor Drain 2: track 5.11 -> 6.62 mm
Other:
- board text added: "+"
- board text added: "-"

Commit message: please please i need to order this
Parts:
- removed C1: .1 uF, Capacitor_SMD:C_0603_1608Metric
- removed C2: 2.2 nF, Capacitor_SMD:C_0603_1608Metric
- removed C3: .1uF, Capacitor_SMD:C_0603_1608Metric
- removed C4: 10nF, Capacitor_SMD:C_0603_1608Metric
- removed U1: MPU-6050, Sensor_Motion:InvenSense_QFN-24_4x4mm_P0.5mm
- added C15: 100 nF, Capacitor_SMD:C_0603_1608Metric, F.Cu at (96.5, 71.0)
- added C16: 100 nF, Capacitor_SMD:C_0603_1608Metric, F.Cu at (99.2, 71.0)
- added U4: LSM6DSM, Package_LGA:LGA-14_3x2.5mm_P0.5mm_LayoutBorder3x4y, F.Cu at (97.8, 67.8)
- R5, R6: value 2.2k -> 4.7 k
- moved C7 11.1 mm to (61.2, 86.2)
- turned L1 to 90 degrees
Connections:
- A2 pad 13: unconnected-(A2-D10-Pad13) -> LSM_CS
- A2 pad 5: unconnected-(A2-D2-Pad5) -> LSM_INT1
Routing:
- net LSM_CS: track 0.00 -> 40.1 mm, vias 0 -> 2
- net V_BAT: track 55.4 -> 24.1 mm, vias 0 -> 1
- net LSM_INT1: track 0.00 -> 24.1 mm, vias 0 -> 2
- net Net-(U3-SW): track 28.5 -> 10.8 mm
- net +3V3: track 165.9 -> 159.2 mm, vias 5 -> 7
- net SCL: track 150.7 -> 146.1 mm
- net Net-(U1-REGOUT): track 2.20 -> 0.00 mm
- net Net-(U1-CPOUT): track 2.07 -> 0.00 mm
- net SDA: track 163.1 -> 161.1 mm
- net CH1: track 36.4 -> 38.0 mm
- net GND: vias 17 -> 36

Commit message: drone_prototype_2
Routing:
- net +3V3: track 159.2 -> 162.6 mm
- net unconnected-(U4-OCS_Aux-Pad10): track 0.00 -> 2.21 mm
- net unconnected-(U4-SDO_Aux-Pad11): track 0.00 -> 1.96 mm
- net unconnected-(U4-INT2-Pad9): track 0.00 -> 1.96 mm
- net unconnected-(U4-SDX-Pad2): track 0.00 -> 1.38 mm
- net unconnected-(U4-SCX-Pad3): track 0.00 -> 1.28 mm
- net unconnected-(U4-SDO/SA0-Pad1): track 0.00 -> 1.13 mm
Changed lines of the file:
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@@
 	)
 	(via
-		(at 100 67.5)
+		(at 100 67.25)
 		(size 0.6)
 		(drill 0.3)
@@
 	)
 	(via
-		(at 95.5 68)
+		(at 95.008106 68.25)
 		(size 0.6)
 		(drill 0.3)
@@
 	)
 	(segment
+		(start 97.275 71)
+		(end 98.475 71)
+		(width 0.3)
+		(layer "F.Cu")
+		(net 8)
+	)
+	(segment
 		(start 94.425 90)
 		(end 93.6 90)
@@
 	)
 	(segment
+		(start 98.475 71)
+		(end 99.25 70.225)
+		(width 0.3)
+		(layer "F.Cu")
+		(net 8)
+	)
+	(segment
 		(start 93.75 75.25)
 		(end 93.75 77.25)
@@
 	)
 	(segment
+		(start 96.5 70.225)
+		(end 97.275 71)
+		(width 0.3)
+		(layer "F.Cu")
+		(net 8)
+	)
+	(segment
 		(start 101.175 76.675)
 		(end 101.175 77.585)
@@
 		(net 46)
 	)
+	(segment
+		(start 96.675 67.5)
+		(end 96 67.5)
+		(width 0.2)
+		(layer "F.Cu")
+		(net 48)
+	)
+	(segment
+		(start 96 67.5)
+		(end 95.5 67)
+		(width 0.2)
+		(layer "F.Cu")
+		(net 48)
+	)
+	(segment
+		(start 95.5 67.75)
+		(end 95.75 68)
+		(width 0.2)
+		(layer "F.Cu")
+		(net 49)
+	)
+	(segment
+		(start 95.75 68)
+		(end 96.675 68)
+		(width 0.2)
+		(layer "F.Cu")
+		(net 49)
+	)
+	(segment
+		(start 96.675 67)
+		(end 96.25 67)
+		(width 0.2)
+		(layer "F.Cu")
+		(net 50)
+	)
+	(segment
+		(start 96.25 67)
+		(end 95.75 66.5)
+		(width 0.2)
+		(layer "F.Cu")
+		(net 50)
+	)
+	(segment
+		(start 99.5 67.5)
+		(end 100 68)
+		(width 0.2)
+		(layer "F.Cu")
+		(net 51)
+	)
+	(segment
+		(start 100 68)
+		(end 101 68)
+		(width 0.2)
+		(layer "F.Cu")
+		(net 51)
+	)
+	(segment
+		(start 99 67.5)
+		(end 99.5 67.5)
+		(width 0.2)
+		(layer "F.Cu")
+		(net 51)
+	)
+	(segment
+		(start 99.75 66.5)
+		(end 100.75 66.5)
+		(width 0.2)
+		(layer "F.Cu")
+		(net 52)
+	)
+	(segment
+		(start 99.5 66.5)
+		(end 99.75 66.5)
+		(width 0.2)
+		(layer "F.Cu")
+		(net 52)
+	)
+	(segment
+		(start 99 67)
+		(end 99.5 66.5)
+		(width 0.2)
+		(layer "F.Cu")
+		(net 52)
+	)
+	(segment
+		(start 100 68.5)
+		(end 100.75 68.5)
+		(width 0.2)
+		(layer "F.Cu")
+		(net 53)
+	)
+	(segment
+		(start 99 68)
+		(end 99.5 68)
+		(width 0.2)
+		(layer "F.Cu")
+		(net 53)
+	)
+	(segment
+		(start 99.5 68)
+		(end 100 68.5)
+		(width 0.2)
+		(layer "F.Cu")
+		(net 53)
+	)
 	(zone
