File: kicad_proj1st/kicad_proj1st.kicad_sch (KiCad schematic)
At the start: 41 parts, among them J1 Conn_01x02, J2 Conn_01x05, J3 Conn_01x02, J4 Conn_01x02, J5 Conn_01x02, J6 Conn_01x02, J7 Conn_01x06, Q1 TSM2302CX, Q2 TSM2302CX, Q3 TSM2302CX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

Commit message: Prototype 2 fin?
Parts:
- C5: value .1uC -> .1uF
- C6: value 4.7uC -> 4.7uF
Changed lines of the file:
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@@
 			)
 		)
-		(property "Value" "4.7uC"
+		(property "Value" "4.7uF"
 			(at 270.51 33.0199 0)
 			(effects
@@
 			)
 		)
-		(property "Value" ".1uC"
+		(property "Value" ".1uF"
 			(at 257.81 33.0199 0)
 			(effects

Commit message: update
Parts:
- added J8: Conn_01x01, Connector_PinHeader_2.54mm:PinHeader_1x01_P2.54mm_Vertical, symbol Connector_Generic:Conn_01x01
Connections:
- net GND: now also J8.1 (Pin_1)
Changed lines of the file:
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@@
+	(symbol
+		(lib_id "power:GND")
+		(at 111.76 90.17 270)
+		(unit 1)
+		(exclude_from_sim no)
+		(in_bom yes)
+		(on_board yes)
+		(dnp no)
+		(fields_autoplaced yes)
+		(property "Reference" "#PWR027"
+			(at 105.41 90.17 0)
+			(effects
+				(font
+					(size 1.27 1.27)
+				)
+				(hide yes)
+			)
+		)
+		(property "Value" "GND"
+			(at 107.95 90.1699 90)
+			(effects
+				(font
+					(size 1.27 1.27)
+				)
+				(justify right)
+			)
+		)
+		(property "Footprint" ""
+			(at 111.76 90.17 0)
+			(effects
+				(font
+					(size 1.27 1.27)
+				)
+				(hide yes)
+			)
+		)
+		(property "Datasheet" ""
+			(at 111.76 90.17 0)
+			(effects
+				(font
+					(size 1.27 1.27)
+				)
+				(hide yes)
+			)
+		)
+		(property "Description" "Power symbol creates a global label with name \"GND\" , ground"
+			(at 111.76 90.17 0)
+			(effects
+				(font
+					(size 1.27 1.27)
+				)
+				(hide yes)
+			)
+		)
+		(pin "1"
+		)
+		(instances
+			(project "kicad_proj1st"
+				(path "/1fefd4af-57a8-41f0-b243-cdbdf510e530"
+					(reference "#PWR027")
+					(unit 1)
+				)
+			)
+		)
+	)
 	(symbol
 		(lib_id "power:GND")
@@
 					(unit 1)
 				)
+			)
+		)
+	)
+	(symbol
+		(lib_id "Connector_Generic:Conn_01x01")
+		(at 116.84 90.17 0)
+		(unit 1)
+		(exclude_from_sim no)
+		(in_bom yes)
+		(on_board yes)
+		(dnp no)
+		(fields_autoplaced yes)
+		(property "Reference" "J8"
+			(at 119.38 88.8999 0)
+			(effects
+				(font
+					(size 1.27 1.27)
+				)
+				(justify left)
+			)
+		)
+		(property "Value" "Conn_01x01"
+			(at 119.38 91.4399 0)
+			(effects
+				(font
+					(size 1.27 1.27)
+				)
+				(justify left)
+			)
+		)
+		(property "Footprint" "Connector_PinHeader_2.54mm:PinHeader_1x01_P2.54mm_Vertical"
+			(at 116.84 90.17 0)
+			(effects
+				(font
+					(size 1.27 1.27)
+				)
+				(hide yes)
+			)
+		)
+		(property "Datasheet" "~"
+			(at 116.84 90.17 0)
+			(effects
+				(font
+					(size 1.27 1.27)
+				)
+				(hide yes)
+			)
+		)
+		(property "Description" "Generic connector, single row, 01x01, script generated (kicad-library-utils/schlib/autogen/connector/)"
+			(at 116.84 90.17 0)
+			(effects
+				(font
+					(size 1.27 1.27)
+				)
+				(hide yes)
+			)
+		)
+		(pin "1"
+		)
+		(instances
+			(project ""
+				(path "/1fefd4af-57a8-41f0-b243-cdbdf510e530"
+					(reference "J8")
+					(unit 1)
+				)

Commit message: please please i need to order this
Parts:
- removed C1: .1 uF, Capacitor_SMD:C_0603_1608Metric, symbol Device:C
- removed C2: 2.2 nF, Capacitor_SMD:C_0603_1608Metric, symbol Device:C
- removed C3: .1uF, Capacitor_SMD:C_0603_1608Metric, symbol Device:C
- removed C4: 10nF, Capacitor_SMD:C_0603_1608Metric, symbol Device:C
- removed U1: MPU-6050, Sensor_Motion:InvenSense_QFN-24_4x4mm_P0.5mm, symbol Sensor_Motion:MPU-6050
- added C15, C16: 100 nF, Capacitor_SMD:C_0603_1608Metric, symbol Device:C
- added U4: LSM6DSM, Package_LGA:LGA-14_3x2.5mm_P0.5mm_LayoutBorder3x4y, symbol Sensor_Motion:LSM6DSM
- R5, R6: value 2.2k -> 4.7 k
Connections:
- net +3V3: now also C15.1, C16.2, U4.5 (VDDIO), U4.8 (VDD)
- net GND: now also C15.2, C16.1, U4.6 (GND), U4.7 (GND)
- net SCL: now also U4.13 (SCL)
- net SDA: now also U4.14 (SDA)
- net LSM_CS: now reaches A2.13 (D10)
- net LSM_CS: now also U4.12 (CS)
- net LSM_INT1: now reaches A2.5 (D2)
- net LSM_INT1: now also U4.4 (INT1)
- no-connect marks 2 -> 0
Other:
- moved on the sheet: R5, R6
